File: kicad/SDP/SDP.kicad_sch (KiCad schematic)
At the start: 64 parts

Commit message: Added GPIO headers, separated power PCB
Parts:
- added D? (x2): Green, symbol Device:LED_Small
- added J?: GPIO, symbol Connector_Generic:Conn_02x12_Top_Bottom
- added J?: UART, symbol Connector_Generic:Conn_02x04_Top_Bottom
- added J?: I2C, symbol Connector_Generic:Conn_02x02_Top_Bottom
- added J?: SPI, symbol Connector_Generic:Conn_02x04_Top_Bottom
- added R?: 2k, symbol Device:R_Small
- added R?: 1k, symbol Device:R_Small
Connections:
- net +12V: now also C?.1, C?.1, FB?.2, R?.1, R?.1, U?.2 (VIN), U?.2 (VIN); no longer F?.1
- net +3V3: now also D?.2 (A)
- net GND: now also R?.2, R?.2
- net P56_SDA1: now also J?.1 (Pin_1)
- net P57_SCL1: now also J?.2 (Pin_2)
- net P58_SCL2: now also J?.4 (Pin_4)
- net P59_SDA2: now also J?.3 (Pin_3)
- net V_IN: now also F?.1; no longer C?.1, C?.1, FB?.2, R?.1, R?.1, U?.2 (VIN), U?.2 (VIN)
- net P1_RG15: now reaches U?.1 (RG15)
- net P1_RG15: now also J?.12 (Pin_12)
- net P10_SCK2: now reaches U?.10 (PMA5/SCK2/CN8/RG6)
- net P10_SCK2: now also J?.8 (Pin_8)
- net P100_RE4: now reaches U?.100 (PMD4/RE4)
- net P100_RE4: now also J?.19 (Pin_19)
- net P11_SDI2: now reaches U?.11 (PMA4/SDI2/CN9/RG7)
- net P11_SDI2: now also J?.7 (Pin_7)
- net P12_SDO2: now reaches U?.12 (PMA3/SDO2/CN10/RG8)
- net P12_SDO2: now also J?.6 (Pin_6)
- net P14_SS2: now reaches U?.14 (PMA2/*SS2/CN11/RG9)
- net P14_SS2: now also J?.5 (Pin_5)
- net P18_RE8: now reaches U?.18 (INT1/RE8)
- net P18_RE8: now also J?.23 (Pin_23)
- net P19_RE9: now reaches U?.19 (INT2/RE9)
- net P19_RE9: now also J?.24 (Pin_24)
- net P20_RB5: now reaches U?.20 (C1IN+/AN5/CN7/RB5)
- net P20_RB5: now also J?.2 (Pin_2)
- net P21_RB4: now reaches U?.21 (C1IN-/AN4/CN6/RB4)
- net P21_RB4: now also J?.1 (Pin_1)
- net P23_SS1: now reaches U?.23 (C2IN-/AN2/*SS1/CN4/RB2)
- net P23_SS1: now also J?.1 (Pin_1)
- net P3_RE5: now reaches U?.3 (PMD5/RE5)
- net P3_RE5: now also J?.20 (Pin_20)
- net P32_TOF1_CE: now reaches U?.32 (C1OUT/AN8/RB8)
- net P33_TOF2_CE: now reaches U?.33 (C2OUT/AN9/RB9)
- net P34_TOF3_CE: now reaches U?.34 (PMA13/CVREF/AN10/RB10)
- net P35_TOF4_CE: now reaches U?.35 (PMA12/AN11/RB11)
- net P39_U2RTS: now reaches U?.39 (*U2RTS/BCLK2/RF13)
- net P39_U2RTS: now also J?.7 (Pin_7)
- net P4_RE6: now reaches U?.4 (PMD6/RE6)
- net P4_RE6: now also J?.21 (Pin_21)
- net P40_U2CTS: now reaches U?.40 (*U2CTS/RF12)
- net P40_U2CTS: now also J?.8 (Pin_8)
- net P41_TOF1_GPIO1: now reaches U?.41 (PMA11/AN12/RB12)
- net P42_TOF2_GPIO1: now reaches U?.42 (PMA10/AN13/RB13)
- net P43_TOF3_GPIO1: now reaches U?.43 (PMA1/AN14/RB14)
- net P44_TOF4_GPIO1: now reaches U?.44 (PMA0/AN15/OCFB/CN12/RB15)
- net P47_U1CTS: now reaches U?.47 (*U1CTS/CN20/RD14)
- net P47_U1CTS: now also J?.4 (Pin_4)
- net P48_U1RTS: now reaches U?.48 (*U1RTS/BCLK1/CN21/RD15)
- net P48_U1RTS: now also J?.3 (Pin_3)
- net P5_RE7: now reaches U?.5 (PMD7/RE7)
- net P5_RE7: now also J?.22 (Pin_22)
- net P53_SDO1: now reaches U?.53 (SDO1/RF8)
- net P53_SDO1: now also J?.2 (Pin_2)
- net P54_SDI1: now reaches U?.54 (SDI1/RF7)
- net P54_SDI1: now also J?.3 (Pin_3)
- net P55_SCK1: now reaches U?.55 (SCK1/INT0/RF6)
- net P55_SCK1: now also J?.4 (Pin_4)
- net P66_RA14: now reaches U?.66 (INT3/RA14)
- net P66_RA14: now also J?.13 (Pin_13)
- net P67_RA15: now reaches U?.67 (INT4/RA15)
- net P67_RA15: now also J?.14 (Pin_14)
- net P68_RD8: now reaches U?.68 (IC1/RTCC/RD8)
- net P68_RD8: now also J?.3 (Pin_3)
- net P69_RD9: now reaches U?.69 (IC2/RD9)
- net P69_RD9: now also J?.4 (Pin_4)
- net P70_RD10: now reaches U?.70 (IC3/PMCS2/RD10)
- net P70_RD10: now also J?.5 (Pin_5)
- net P71_RD11: now reaches U?.71 (IC4/PMCS1/RD11)
- net P71_RD11: now also J?.6 (Pin_6)
- net P89_RG1: now reaches U?.89 (RG1)
- net P89_RG1: now also J?.8 (Pin_8)
- net P90_RG0: now reaches U?.90 (RG0)
- net P90_RG0: now also J?.7 (Pin_7)
- net P92_TEMP2: now reaches U?.92 (RA7)
- net P93_RE0: now reaches U?.93 (PMD0/RE0)
- net P93_RE0: now also J?.15 (Pin_15)
- net P94_RE1: now reaches U?.94 (PMD1/RE1)
- net P94_RE1: now also J?.16 (Pin_16)
- net P98_RE2: now reaches U?.98 (PMD2/RE2)
- net P98_RE2: now also J?.17 (Pin_17)
- net P99_RE3: now reaches U?.99 (PMD3/RE3)
- net P99_RE3: now also J?.18 (Pin_18)
- net P51_U1TX: now reaches U?.51 (U1TX/RF3)
- net P51_U1TX: now also J?.5 (Pin_5)
- net P52_U1RX: now reaches U?.52 (U1RX/RF2)
- net P52_U1RX: now also J?.6 (Pin_6)
- net P16_LED: now reaches U?.61 (TDO/RA5)
- net P16_LED: now also D?.2 (A)
- net P49_BT_RX renamed P49_U2RX
- net P49_U2RX: now also J?.2 (Pin_2)
- net P50_BT_TX renamed P50_U2TX
- net P50_U2TX: now also J?.1 (Pin_1)
- net P91_TEMP renamed P91_TEMP1
- net P95_TOF1_CE renamed P95_RG14
- net P95_RG14: now also J?.11 (Pin_11)
- net P96_TOF2_CE renamed P96_RG12
- net P96_RG12: now also J?.9 (Pin_9)
- net P97_TOF3_CE renamed P97_RG13
- net P97_RG13: now also J?.10 (Pin_10)
- new net: D?.1 (K), R?.1 (x2)
Other:
- moved on the sheet: BT?, C?, D?, F?, FB?, J?, L?, MOSFET?, R?, U?, U?C

Commit message: Part selection
Parts:
- gave numbers to parts that had none: 6
