File: kicad/SDP/watersubsystem.kicad_sch (KiCad schematic)
At the start: 15 parts, among them J15 Conn_01x02, J16 Conn_01x02, J23 Conn_01x02, Q1 IRLZ44N, Q2 IRLZ44N, Q3 IRLZ44N

Commit message: Assigned footprints and removed ferrite bead
Parts:
- C28, C29, C36: footprint (none) -> Capacitor_THT:C_Radial_D12.5mm_H20.0mm_P5.00mm
Changed lines of the file:
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@@
       (effects (font (size 1.27 1.27)) (justify left))
     )
-    (property "Footprint" "" (id 2) (at 74.422 56.388 0)
+    (property "Footprint" "Capacitor_THT:C_Radial_D12.5mm_H20.0mm_P5.00mm" (id 2) (at 74.422 56.388 0)
       (effects (font (size 1.27 1.27)) hide)
     )
@@
       (effects (font (size 1.27 1.27)) (justify left))
     )
-    (property "Footprint" "" (id 2) (at 141.732 56.642 0)
+    (property "Footprint" "Capacitor_THT:C_Radial_D12.5mm_H20.0mm_P5.00mm" (id 2) (at 141.732 56.642 0)
       (effects (font (size 1.27 1.27)) hide)
     )
@@
       (effects (font (size 1.27 1.27)) (justify left))
     )
-    (property "Footprint" "" (id 2) (at 75.438 117.856 0)
+    (property "Footprint" "Capacitor_THT:C_Radial_D12.5mm_H20.0mm_P5.00mm" (id 2) (at 75.438 117.856 0)
       (effects (font (size 1.27 1.27)) hide)
     )

Commit message: PCB layout and schematic updates
Parts:
- D6, D7, D8: value 1N4007 -> SS1200; footprint Diode_THT:D_DO-41_SOD81_P10.16mm_Horizontal -> Diode_SMD:D_SMA
- Q1, Q2, Q3: footprint Package_TO_SOT_THT:TO-220-3_Vertical -> Package_TO_SOT_SMD:TO-263-2
Changed lines of the file:
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@@
   (symbol (lib_id "Diode:1N4007") (at 129.032 49.022 270) (unit 1)
     (in_bom yes) (on_board yes) (fields_autoplaced)
-    (property "Reference" "D7" (id 0) (at 131.572 47.7519 90)
+    (property "Reference" "D7" (id 0) (at 132.08 47.7519 90)
       (effects (font (size 1.27 1.27)) (justify left))
     )
-    (property "Value" "1N4007" (id 1) (at 131.572 50.2919 90)
+    (property "Value" "SS1200" (id 1) (at 132.08 50.2919 90)
       (effects (font (size 1.27 1.27)) (justify left))
     )
-    (property "Footprint" "Diode_THT:D_DO-41_SOD81_P10.16mm_Horizontal" (id 2) (at 124.587 49.022 0)
+    (property "Footprint" "Diode_SMD:D_SMA" (id 2) (at 124.587 49.022 0)
       (effects (font (size 1.27 1.27)) hide)
     )
@@
       (effects (font (size 1.27 1.27)) (justify left))
     )
-    (property "Footprint" "Package_TO_SOT_THT:TO-220-3_Vertical" (id 2) (at 59.182 64.643 0)
+    (property "Footprint" "Package_TO_SOT_SMD:TO-263-2" (id 2) (at 59.182 64.643 0)
       (effects (font (size 1.27 1.27) italic) (justify left) hide)
     )
@@
       (effects (font (size 1.27 1.27)) (justify left))
     )
-    (property "Footprint" "Package_TO_SOT_THT:TO-220-3_Vertical" (id 2) (at 126.492 64.897 0)
+    (property "Footprint" "Package_TO_SOT_SMD:TO-263-2" (id 2) (at 126.492 64.897 0)
       (effects (font (size 1.27 1.27) italic) (justify left) hide)
     )
@@
       (effects (font (size 1.27 1.27)) (justify left))
     )
-    (property "Footprint" "Package_TO_SOT_THT:TO-220-3_Vertical" (id 2) (at 60.198 126.111 0)
+    (property "Footprint" "Package_TO_SOT_SMD:TO-263-2" (id 2) (at 60.198 126.111 0)
       (effects (font (size 1.27 1.27) italic) (justify left) hide)
     )
@@
   (symbol (lib_id "Diode:1N4007") (at 61.722 48.768 270) (unit 1)
     (in_bom yes) (on_board yes) (fields_autoplaced)
-    (property "Reference" "D6" (id 0) (at 64.262 47.4979 90)
+    (property "Reference" "D6" (id 0) (at 64.77 47.4979 90)
       (effects (font (size 1.27 1.27)) (justify left))
     )
-    (property "Value" "1N4007" (id 1) (at 64.262 50.0379 90)
+    (property "Value" "SS1200" (id 1) (at 64.77 50.0379 90)
       (effects (font (size 1.27 1.27)) (justify left))
     )
-    (property "Footprint" "Diode_THT:D_DO-41_SOD81_P10.16mm_Horizontal" (id 2) (at 57.277 48.768 0)
+    (property "Footprint" "Diode_SMD:D_SMA" (id 2) (at 57.277 48.768 0)
       (effects (font (size 1.27 1.27)) hide)
     )
@@
   (symbol (lib_id "Diode:1N4007") (at 62.738 110.236 270) (unit 1)
     (in_bom yes) (on_board yes) (fields_autoplaced)
-    (property "Reference" "D8" (id 0) (at 65.278 108.9659 90)
+    (property "Reference" "D8" (id 0) (at 64.77 108.9659 90)
       (effects (font (size 1.27 1.27)) (justify left))
     )
-    (property "Value" "1N4007" (id 1) (at 65.278 111.5059 90)
+    (property "Value" "SS1200" (id 1) (at 64.77 111.5059 90)
       (effects (font (size 1.27 1.27)) (justify left))
     )
-    (property "Footprint" "Diode_THT:D_DO-41_SOD81_P10.16mm_Horizontal" (id 2) (at 58.293 110.236 0)
+    (property "Footprint" "Diode_SMD:D_SMA" (id 2) (at 58.293 110.236 0)
       (effects (font (size 1.27 1.27)) hide)
     )
