File: kicad/SDP/SDP.kicad_pcb (KiCad board)
At the start: 4 copper layers, 98 x 98 mm, 105 parts, among them J1 GPIO, J10 Limit, J11 Conn_01x07, J12 Conn_01x07, J13 Conn_01x03, J14 Conn_01x03, J15 Conn_01x03, J16 Conn_01x03, J17 Conn_01x03, J18 12V, J19 I2C2, J2 Conn_01x03, J20 POWER, J24 POWER, J25 Conn_01x04, J26 Conn_01x02, J27 MOTOR, J3 UART, J4 I2C1, J5 Conn_01x04, J6 Conn_01x04, J7 RJ25, J8 Conn_01x07, J9 Conn_01x07, SW1 SW_Push_Dual, U1 TPS54233, U2 TPS54233, U3 PIC24FJ128GA010-I/PT, U4 DS3231SN-T&R, Y1 8MHz, Y2 32.768kHz

Commit message: Final PCB layout changes
Connections:
- J27 pad 15: GND -> unconnected-(J27-Pad15)
Routing:
- net Net-(D2-Pad1): track 13.2 -> 0.00 mm
- net +3V3: track 123.1 -> 113.9 mm, vias 49 -> 42
- net +12V: track 83.4 -> 89.9 mm
- net P52_U1RX: track 77.2 -> 77.8 mm
- net GND: vias 97 -> 99
Other:
- board text added: "+"
- board text added: "12V"
- board text added: "JLCJLCJLCJLC"
- board text added: "LIMIT"
- board text added: "MOTOR"
- board text added: "POWER"
- board text added: "PROXIMITY"
- board text added: "RESET"
- board text removed: "Limit"
- board text removed: "Motor"
- board text removed: "Power"
- board text removed: "Proximity"
