File: kicad/SDP_motors/SDP_motors.kicad_sch (KiCad schematic)
At the start: 69 parts, among them J1 Conn_01x04, J2 Conn_01x04, J3 Conn_01x04, J4 Conn_01x04, J5 Conn_01x04, J6 Conn_01x04, J7 Conn_01x02, J8 Conn_01x02, J9 Conn_01x02, Q1 IRLZ44N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

Commit message: Added proximity sensor headers
Parts:
- added H1, H2, H3, H4: MountingHole_Pad, MountingHole:MountingHole_3.2mm_M3_Pad, symbol Mechanical:MountingHole_Pad
- added J10: MOTOR, Connector_PinSocket_2.54mm:PinSocket_2x08_P2.54mm_Vertical, symbol Connector_Generic:Conn_02x08_Odd_Even
- added TP1, TP2, TP3, TP4: TestPoint_Small, TestPoint:TestPoint_Pad_D2.0mm, symbol Connector:TestPoint_Small
Connections:
- net +12V: now also J10.15 (Pin_15)
- net +3V3: now also J10.1 (Pin_1), J10.2 (Pin_2), TP1.1, TP2.1
- net GND: now also H1.1, H2.1, H3.1, H4.1, J10.16 (Pin_16), TP3.1, TP4.1
- net P72_FAN: now also J10.3 (Pin_3)
- net P76_EN: now also J10.4 (Pin_4)
- net P77_STEP: now also J10.5 (Pin_5)
- net P78_DIR: now also J10.6 (Pin_6)
- net P79_EN: now also J10.7 (Pin_7)
- net P80_STEP: now also J10.8 (Pin_8)
- net P81_DIR: now also J10.9 (Pin_9)
- net P82_EN: now also J10.10 (Pin_10)
- net P83_STEP: now also J10.11 (Pin_11)
- net P84_DIR: now also J10.12 (Pin_12)
- net P87_MTR1: now also J10.13 (Pin_13)
- net P88_MTR2: now also J10.14 (Pin_14)
